Commit message: driving bot around

File: description/robot.urdf.xacro (robot description, xacro)
@@ -2,3 +2,4 @@
 <robot xmlns:xacro="http://www.ros.org/wiki/xacro"  name="robot">
 <xacro:include filename="robot_core.xacro" />
+<xacro:include filename="gazebo_control.xacro"/>
 </robot>

File: description/robot_core.xacro (robot description, xacro)
@@ -57,5 +57,5 @@
         <visual>
             <geometry>
-                <cylinder radius="0.1" length="0.07"/>
+                <cylinder radius="0.15" length="0.07"/>
             </geometry>
             <material name="blue"/>
@@ -63,8 +63,8 @@
         <collision>
             <geometry>
-                <cylinder radius="0.1" length="0.07"/>
+                <cylinder radius="0.15" length="0.07"/>
             </geometry>
         </collision>
-        <xacro:inertial_cylinder mass="10" length="0.07" radius="0.1">
+        <xacro:inertial_cylinder mass="10" length="0.07" radius="0.15">
             <origin xyz="0 0 0" rpy="0 0 0"/>
         </xacro:inertial_cylinder>
@@ -83,5 +83,5 @@
         <visual>
             <geometry>
-                <cylinder radius="0.1" length="0.07"/>
+                <cylinder radius="0.15" length="0.07"/>
             </geometry>
             <material name="blue"/>
@@ -89,8 +89,8 @@
         <collision>
             <geometry>
-                <cylinder radius="0.1" length="0.07"/>
+                <cylinder radius="0.15" length="0.07"/>
             </geometry>
         </collision>
-        <xacro:inertial_cylinder mass="10" length="0.07" radius="0.1">
+        <xacro:inertial_cylinder mass="10" length="0.07" radius="0.15">
             <origin xyz="0 0 0" rpy="0 0 0"/>
         </xacro:inertial_cylinder>
@@ -108,5 +108,5 @@
         <visual>
             <geometry>
-                <sphere radius="0.1"/>
+                <sphere radius="0.14"/>
             </geometry>
             <material name="black"/>
@@ -114,8 +114,8 @@
         <collision>
             <geometry>
-                <sphere radius="0.1"/>
+                <sphere radius="0.14"/>
             </geometry>
         </collision>
-        <xacro:inertial_sphere mass="5" radius="0.1">
+        <xacro:inertial_sphere mass="5" radius="0.14">
             <origin xyz="0 0 0" rpy="0 0 0"/>
         </xacro:inertial_sphere>
@@ -135,5 +135,5 @@
         <visual>
             <geometry>
-                <sphere radius="0.1"/>
+                <sphere radius="0.14"/>
             </geometry>
             <material name="black"/>
@@ -141,8 +141,8 @@
         <collision>
             <geometry>
-                <sphere radius="0.1"/>
+                <sphere radius="0.14"/>
             </geometry>
         </collision>
-        <xacro:inertial_sphere mass="5" radius="0.1">
+        <xacro:inertial_sphere mass="5" radius="0.14">
             <origin xyz="0 0 0" rpy="0 0 0"/>
         </xacro:inertial_sphere>

Commit message: lidar davamate

File: description/robot.urdf.xacro (robot description, xacro)
@@ -3,3 +3,4 @@
 <xacro:include filename="robot_core.xacro" />
 <xacro:include filename="gazebo_control.xacro"/>
+<xacro:include filename="lidar.xacro"/>
 </robot>

File: description/robot_core.xacro (robot description, xacro)
@@ -108,5 +108,5 @@
         <visual>
             <geometry>
-                <sphere radius="0.14"/>
+                <sphere radius="0.15"/>
             </geometry>
             <material name="black"/>
@@ -114,8 +114,8 @@
         <collision>
             <geometry>
-                <sphere radius="0.14"/>
+                <sphere radius="0.15"/>
             </geometry>
         </collision>
-        <xacro:inertial_sphere mass="5" radius="0.14">
+        <xacro:inertial_sphere mass="5" radius="0.15">
             <origin xyz="0 0 0" rpy="0 0 0"/>
         </xacro:inertial_sphere>
@@ -135,5 +135,5 @@
         <visual>
             <geometry>
-                <sphere radius="0.14"/>
+                <sphere radius="0.15"/>
             </geometry>
             <material name="black"/>
@@ -141,8 +141,8 @@
         <collision>
             <geometry>
-                <sphere radius="0.14"/>
+                <sphere radius="0.15"/>
             </geometry>
         </collision>
-        <xacro:inertial_sphere mass="5" radius="0.14">
+        <xacro:inertial_sphere mass="5" radius="0.15">
             <origin xyz="0 0 0" rpy="0 0 0"/>
         </xacro:inertial_sphere>
